Commit message: Ship Phase 6 transfer, RoboMaster wall layout, and token tracker.
Align PPO wall-follow with P2_D3 medium standoff, enlarge top-down maze/robot, add Fig. 4 scenario tasks, and expose /tokens so smokes can run on current code.

Co-authored-by: Cursor <cursoragent@cursor.com>

File: robolab/robolab/robots/diffdrive_lidar/robot.urdf (robot description, URDF)
Before this commit: robot diffdrive_lidar, 3 links, 2 joints
Links:
- added link armor_front, mass 0.3; collision box size=0.08 0.36 0.10; visual box size=0.08 0.36 0.10
- link base_link: mass 4.0 -> 8.0; geometry collision box size=0.55 0.42 0.12; visual box size=0.55 0.42 0.12
- link left_wheel: mass 0.4 -> 0.6; geometry collision cylinder length=0.06 radius=0.075; visual cylinder length=0.06 radius=0.075
- link right_wheel: mass 0.4 -> 0.6; geometry collision cylinder length=0.06 radius=0.075; visual cylinder length=0.06 radius=0.075
Joints:
- added joint armor_front_joint: type fixed, parent base_link, child armor_front, origin xyz=0.24 0 0.12 rpy=0 0 0
- joint left_wheel_joint: origin xyz=0 0.14 0.05 rpy=0 0 0 -> xyz=0 0.22 0.075 rpy=0 0 0
- joint right_wheel_joint: origin xyz=0 -0.14 0.05 rpy=0 0 0 -> xyz=0 -0.22 0.075 rpy=0 0 0
